File: RP2350B_Consol.kicad_sch (KiCad schematic)
At the start: 33 parts, among them J1 Conn_01x15_Socket, J10 VGA, J2 Conn_01x15_Socket, J3 Conn_01x15_Socket, J4 Conn_01x15_Socket, J5 Conn_02x06_Odd_Even, J6 Conn_02x20_Odd_Even, J7 NES_Joystick1, J8 NES_Joystick2, J9 PJ320D, U2 SN76489AN

Commit message: Update RP2350B_Consol.kicad_sch
Parts:
- DD1: footprint PicoSegaLibrary:RP2040_purple_allPin -> Library:RP2040_purple_allPin
- J9: footprint PicoSegaLibrary:PJ320D_3.5mm_Jack -> Library:PJ320D_3.5mm_Jack
Changed lines of the file:
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@@
 			)
 		)
-		(property "Footprint" "PicoSegaLibrary:PJ320D_3.5mm_Jack"
+		(property "Footprint" "Library:PJ320D_3.5mm_Jack"
 			(at 187.706 224.282 0)
 			(effects
@@
 			)
 		)
-		(property "Footprint" "PicoSegaLibrary:RP2040_purple_allPin"
+		(property "Footprint" "Library:RP2040_purple_allPin"
 			(at 279.4 177.8 0)
 			(effects
