File: MOC6502.kicad_sch (KiCad schematic)
At the start: 8 parts, among them J11 Conn_02x06_Odd_Even, J12 Conn_02x20_Odd_Even, SW2 "RESET"

Commit message: Update MOC6502.kicad_sch
Parts:
- removed J11: Conn_02x06_Odd_Even, UM6502:EDGE_2x12, symbol Connector_Generic:Conn_02x06_Odd_Even
- added J18: Conn_02x10_Odd_Even, Library:EDGE_2x10, symbol Connector_Generic:Conn_02x10_Odd_Even
- J12: footprint UM6502:EDGE_2x20 -> Library:EDGE_2x20
- SW2: footprint (none) -> Button_Switch_THT:SW_Tactile_SPST_Angled_PTS645Vx31-2LFS
Connections:
- net CLK_2MHz: now also J18.4 (Pin_4)
- net GND1: now also J18.1 (Pin_1), J18.2 (Pin_2)
- net ~{RESETM}: now also J18.10 (Pin_10); no longer J12.3 (Pin_3)
- net CLK6502: now reaches J12.9 (Pin_9)
- net CLK6502: now also U3.37 (F0(IN))
- net CLK: no longer names the net of J12.7 (Pin_7)
- net CLK: no longer U3.37 (F0(IN))
Other:
- moved on the sheet: J12
