File: RP2350B_Consol.kicad_pcb (KiCad board)
At the start: 2 copper layers, 35 parts, among them J1 Conn_01x15_Socket, J10 VGA, J2 Conn_01x15_Socket, J3 Conn_01x15_Socket, J4 Conn_01x15_Socket, J7 NES_Joystick1, J8 NES_Joystick2, U2 SN76489AN, U4 Z80CPU

Commit message: Update RP2350B_Consol.kicad_pcb
Parts:
- removed D1: D, Diode_SMD:D_1206_3216Metric_Pad1.42x1.75mm_HandSolder
- added ?: , , F.Cu at (343.0, 85.1)
- added ?: , , F.Cu at (288.5, 100.3)
- added ?: , , F.Cu at (177.8, 135.9)
- added ?: , , F.Cu at (170.2, 148.6)
- added ?: , , F.Cu at (340.4, 87.6)
- added ?: , , F.Cu at (340.4, 107.9)
- added ?: , , F.Cu at (301.2, 105.4)
- added ?: , , F.Cu at (296.1, 100.3)
- added ?: , , F.Cu at (172.7, 151.1)
- added ?: , , F.Cu at (170.2, 135.9)
- added ?: , , F.Cu at (288.5, 80.0)
- added ?: , , F.Cu at (345.5, 97.8)
- added ?: , , F.Cu at (301.2, 100.3)
- added ?: , , F.Cu at (340.4, 92.7)
- added ?: , , F.Cu at (301.2, 92.7)
- added ?: , , F.Cu at (332.8, 102.8)
- added ?: , , F.Cu at (303.8, 105.4)
- added ?: , , F.Cu at (288.5, 92.7)
- added ?: , , F.Cu at (330.3, 100.3)
- added ?: , , F.Cu at (170.2, 141.0)
- added ?: , , F.Cu at (291.1, 85.1)
- added ?: , , F.Cu at (337.9, 105.4)
- added ?: , , F.Cu at (301.2, 90.1)
- added ?: , , F.Cu at (337.9, 92.7)
- added ?: , , F.Cu at (293.6, 82.5)
- added ?: , , F.Cu at (296.1, 102.8)
- added ?: , , F.Cu at (327.7, 92.7)
- added ?: , , F.Cu at (165.1, 146.1)
- added ?: , , F.Cu at (330.3, 85.1)
- added ?: , , F.Cu at (288.5, 97.8)
- added ?: , , F.Cu at (177.8, 138.4)
- added ?: , , F.Cu at (175.3, 151.1)
- added ?: , , F.Cu at (293.6, 97.8)
- added ?: , , F.Cu at (165.1, 123.2)
- added ?: , , F.Cu at (165.1, 148.6)
- added ?: , , F.Cu at (330.3, 97.8)
- added ?: , , F.Cu at (335.3, 107.9)
- added ?: , , F.Cu at (175.3, 128.3)
- added ?: , , F.Cu at (332.8, 97.8)
- added ?: , , F.Cu at (303.8, 87.6)
- added ?: , , F.Cu at (327.7, 90.1)
- added ?: , , F.Cu at (343.0, 92.7)
- added ?: , , F.Cu at (165.1, 143.5)
- added ?: , , F.Cu at (291.1, 97.8)
- added ?: , , F.Cu at (345.5, 105.4)
- added ?: , , F.Cu at (296.1, 105.4)
- added ?: , , F.Cu at (298.7, 87.6)
- added ?: , , F.Cu at (332.8, 92.7)
- added ?: , , F.Cu at (172.7, 141.0)
- added ?: , , F.Cu at (172.7, 138.4)
- added ?: , , F.Cu at (291.1, 80.0)
- added ?: , , F.Cu at (298.7, 102.8)
- added ?: , , F.Cu at (170.2, 125.7)
- added ?: , , F.Cu at (296.1, 85.1)
- added ?: , , F.Cu at (293.6, 105.4)
- added ?: , , F.Cu at (301.2, 87.6)
- added ?: , , F.Cu at (303.8, 100.3)
- added ?: , , F.Cu at (298.7, 90.1)
- added ?: , , F.Cu at (293.6, 95.2)
- added ?: , , F.Cu at (332.8, 107.9)
- added ?: , , F.Cu at (172.7, 146.1)
- added ?: , , F.Cu at (170.2, 133.3)
- added ?: , , F.Cu at (165.1, 138.4)
- added ?: , , F.Cu at (288.5, 102.8)
- added ?: , , F.Cu at (343.0, 87.6)
- added ?: , , F.Cu at (330.3, 105.4)
- added ?: , , F.Cu at (296.1, 95.2)
- added ?: , , F.Cu at (303.8, 90.1)
- added ?: , , F.Cu at (172.7, 143.5)
- added ?: , , F.Cu at (340.4, 105.4)
- added ?: , , F.Cu at (332.8, 90.1)
- added ?: , , F.Cu at (343.0, 90.1)
- added ?: , , F.Cu at (330.3, 107.9)
- added ?: , , F.Cu at (327.7, 102.8)
- added ?: , , F.Cu at (337.9, 107.9)
- added ?: , , F.Cu at (165.1, 125.7)
- added ?: , , F.Cu at (303.8, 102.8)
- added ?: , , F.Cu at (303.8, 82.5)
- added ?: , , F.Cu at (327.7, 95.2)
- added ?: , , F.Cu at (340.4, 85.1)
- added ?: , , F.Cu at (288.5, 85.1)
- added ?: , , F.Cu at (335.3, 92.7)
- added ?: , , F.Cu at (288.5, 107.9)
- added ?: , , F.Cu at (332.8, 100.3)
- added ?: , , F.Cu at (167.6, 130.8)
- added ?: , , F.Cu at (296.1, 97.8)
- added ?: , , F.Cu at (167.6, 133.3)
- added ?: , , F.Cu at (303.8, 107.9)
- added ?: , , F.Cu at (298.7, 97.8)
- added ?: , , F.Cu at (332.8, 105.4)
- added ?: , , F.Cu at (167.6, 148.6)
- added ?: , , F.Cu at (288.5, 105.4)
- added ?: , , F.Cu at (340.4, 102.8)
- added ?: , , F.Cu at (335.3, 90.1)
- added ?: , , F.Cu at (345.5, 87.6)
- added ?: , , F.Cu at (175.3, 135.9)
- added ?: , , F.Cu at (167.6, 125.7)
- added ?: , , F.Cu at (175.3, 141.0)
- added ?: , , F.Cu at (335.3, 105.4)
- added ?: , , F.Cu at (165.1, 141.0)
- added ?: , , F.Cu at (330.3, 92.7)
- added ?: , , F.Cu at (345.5, 102.8)
- added ?: , , F.Cu at (298.7, 82.5)
- added ?: , , F.Cu at (175.3, 125.7)
- added ?: , , F.Cu at (337.9, 97.8)
- added ?: , , F.Cu at (175.3, 148.6)
- added ?: , , F.Cu at (335.3, 100.3)
- added ?: , , F.Cu at (170.2, 138.4)
- added ?: , , F.Cu at (177.8, 146.1)
- added ?: , , F.Cu at (170.2, 128.3)
- added ?: , , F.Cu at (167.6, 128.3)
- added ?: , , F.Cu at (332.8, 87.6)
- added ?: , , F.Cu at (298.7, 80.0)
- added ?: , , F.Cu at (345.5, 100.3)
- added ?: , , F.Cu at (303.8, 97.8)
- added ?: , , F.Cu at (301.2, 80.0)
- added ?: , , F.Cu at (291.1, 87.6)
- added ?: , , F.Cu at (167.6, 143.5)
- added ?: , , F.Cu at (340.4, 95.2)
- added ?: , , F.Cu at (177.8, 128.3)
- added ?: , , F.Cu at (296.1, 82.5)
- added ?: , , F.Cu at (298.7, 95.2)
- added ?: , , F.Cu at (337.9, 100.3)
- added ?: , , F.Cu at (296.1, 87.6)
- added ?: , , F.Cu at (327.7, 107.9)
- added ?: , , F.Cu at (172.7, 128.3)
- added ?: , , F.Cu at (288.5, 82.5)
- added ?: , , F.Cu at (170.2, 151.1)
- added ?: , , F.Cu at (343.0, 100.3)
- added ?: , , F.Cu at (343.0, 95.2)
- added ?: , , F.Cu at (296.1, 80.0)
- added ?: , , F.Cu at (343.0, 97.8)
- added ?: , , F.Cu at (293.6, 102.8)
- added ?: , , F.Cu at (170.2, 143.5)
- added ?: , , F.Cu at (335.3, 87.6)
- added ?: , , F.Cu at (293.6, 90.1)
- added ?: , , F.Cu at (165.1, 135.9)
- added ?: , , F.Cu at (327.7, 85.1)
- added ?: , , F.Cu at (291.1, 92.7)
- added ?: , , F.Cu at (343.0, 105.4)
- added ?: , , F.Cu at (345.5, 92.7)
- added ?: , , F.Cu at (343.0, 102.8)
- added ?: , , F.Cu at (165.1, 151.1)
- added ?: , , F.Cu at (343.0, 107.9)
- added ?: , , F.Cu at (340.4, 90.1)
- added ?: , , F.Cu at (332.8, 85.1)
- added ?: , , F.Cu at (167.6, 135.9)
- added ?: , , F.Cu at (291.1, 107.9)
- added ?: , , F.Cu at (288.5, 87.6)
- added ?: , , F.Cu at (303.8, 80.0)
- added ?: , , F.Cu at (291.1, 105.4)
- added ?: , , F.Cu at (291.1, 100.3)
- added ?: , , F.Cu at (165.1, 133.3)
- added ?: , , F.Cu at (293.6, 85.1)
- added ?: , , F.Cu at (291.1, 82.5)
- added ?: , , F.Cu at (167.6, 123.2)
- added ?: , , F.Cu at (177.8, 148.6)
- added ?: , , F.Cu at (167.6, 138.4)
- added ?: , , F.Cu at (175.3, 123.2)
- added ?: , , F.Cu at (345.5, 90.1)
- added ?: , , F.Cu at (175.3, 143.5)
- added ?: , , F.Cu at (303.8, 92.7)
- added ?: , , F.Cu at (172.7, 130.8)
- added ?: , , F.Cu at (345.5, 107.9)
- added ?: , , F.Cu at (301.2, 95.2)
- added ?: , , F.Cu at (291.1, 102.8)
- added ?: , , F.Cu at (288.5, 90.1)
- added ?: , , F.Cu at (167.6, 151.1)
- added ?: , , F.Cu at (296.1, 90.1)
- added ?: , , F.Cu at (301.2, 107.9)
- added ?: , , F.Cu at (296.1, 107.9)
- added ?: , , F.Cu at (291.1, 95.2)
- added ?: , , F.Cu at (177.8, 143.5)
- added ?: , , F.Cu at (288.5, 95.2)
- added ?: , , F.Cu at (293.6, 80.0)
- added ?: , , F.Cu at (301.2, 85.1)
- added ?: , , F.Cu at (330.3, 90.1)
- added ?: , , F.Cu at (335.3, 95.2)
- added ?: , , F.Cu at (291.1, 90.1)
- added ?: , , F.Cu at (172.7, 148.6)
- added ?: , , F.Cu at (301.2, 102.8)
- added ?: , , F.Cu at (165.1, 130.8)
- added ?: , , F.Cu at (298.7, 92.7)
- added ?: , , F.Cu at (172.7, 123.2)
- added ?: , , F.Cu at (337.9, 85.1)
- added ?: , , F.Cu at (335.3, 85.1)
- added ?: , , F.Cu at (175.3, 130.8)
- added ?: , , F.Cu at (345.5, 85.1)
- added ?: , , F.Cu at (337.9, 87.6)
- added ?: , , F.Cu at (298.7, 85.1)
- added ?: , , F.Cu at (337.9, 95.2)
- added ?: , , F.Cu at (330.3, 95.2)
- added ?: , , F.Cu at (298.7, 107.9)
- added ?: , , F.Cu at (177.8, 133.3)
- added ?: , , F.Cu at (170.2, 123.2)
- added ?: , , F.Cu at (335.3, 97.8)
- added ?: , , F.Cu at (170.2, 130.8)
- added ?: , , F.Cu at (177.8, 130.8)
- added ?: , , F.Cu at (175.3, 138.4)
- added ?: , , F.Cu at (293.6, 87.6)
- added ?: , , F.Cu at (293.6, 100.3)
- added ?: , , F.Cu at (330.3, 102.8)
- added ?: , , F.Cu at (170.2, 146.1)
- added ?: , , F.Cu at (172.7, 133.3)
- added ?: , , F.Cu at (177.8, 125.7)
- added ?: , , F.Cu at (327.7, 97.8)
- added ?: , , F.Cu at (340.4, 97.8)
- added ?: , , F.Cu at (175.3, 146.1)
- added ?: , , F.Cu at (335.3, 102.8)
- added ?: , , F.Cu at (167.6, 141.0)
- added ?: , , F.Cu at (301.2, 97.8)
- added ?: , , F.Cu at (296.1, 92.7)
- added ?: , , F.Cu at (340.4, 100.3)
- added ?: , , F.Cu at (177.8, 123.2)
- added ?: , , F.Cu at (175.3, 133.3)
- added ?: , , F.Cu at (303.8, 95.2)
- added ?: , , F.Cu at (327.7, 105.4)
- added ?: , , F.Cu at (332.8, 95.2)
- added ?: , , F.Cu at (330.3, 87.6)
- added ?: , , F.Cu at (172.7, 125.7)
- added ?: , , F.Cu at (337.9, 90.1)
- added ?: , , F.Cu at (177.8, 141.0)
- added ?: , , F.Cu at (298.7, 105.4)
- added ?: , , F.Cu at (327.7, 100.3)
- added ?: , , F.Cu at (337.9, 102.8)
- added ?: , , F.Cu at (165.1, 128.3)
- added ?: , , F.Cu at (301.2, 82.5)
- added ?: , , F.Cu at (293.6, 92.7)
- added ?: , , F.Cu at (327.7, 87.6)
- added ?: , , F.Cu at (298.7, 100.3)
- added ?: , , F.Cu at (303.8, 85.1)
- added ?: , , F.Cu at (345.5, 95.2)
- added ?: , , F.Cu at (293.6, 107.9)
- added ?: , , F.Cu at (177.8, 151.1)
- added ?: , , F.Cu at (172.7, 135.9)
- added ?: , , F.Cu at (167.6, 146.1)
- added BZ1: Buzzer, Buzzer_Beeper:Buzzer_12x9.5RM7.6, F.Cu at (397.9, 77.6)
- added C10: 1.0uF, Capacitor_SMD:C_0805_2012Metric_Pad1.18x1.45mm_HandSolder, F.Cu at (51.4, 144.8)
- added C11: 1.0uF, Capacitor_SMD:C_0805_2012Metric_Pad1.18x1.45mm_HandSolder, F.Cu at (48.3, 144.8)
- added C12: 6800, Capacitor_SMD:C_0805_2012Metric_Pad1.18x1.45mm_HandSolder, F.Cu at (251.2, 94.0)
- added C13: 1.0uF, Capacitor_SMD:C_0805_2012Metric_Pad1.18x1.45mm_HandSolder, F.Cu at (256.3, 94.0)
- added C14: 0.1uF, Capacitor_SMD:C_0805_2012Metric_Pad1.18x1.45mm_HandSolder, F.Cu at (256.9, 122.2)
- added C15: 100.0, Capacitor_THT:CP_Radial_D6.3mm_P2.50mm, F.Cu at (397.9, 90.0)
- added C16: 0.1, Capacitor_SMD:C_0805_2012Metric_Pad1.18x1.45mm_HandSolder, F.Cu at (384.3, 98.9)
- added C17: 1.0uF, Capacitor_SMD:C_0805_2012Metric_Pad1.18x1.45mm_HandSolder, F.Cu at (160.0, 87.6)
- added C18: 0.1u, Capacitor_SMD:C_0805_2012Metric_Pad1.18x1.45mm_HandSolder, F.Cu at (66.7, 89.3)
- added C19: 0.022, Capacitor_SMD:C_0805_2012Metric_Pad1.18x1.45mm_HandSolder, F.Cu at (176.5, 104.1)
- added C20: 47.0uF, Capacitor_THT:CP_Radial_D5.0mm_P2.00mm, F.Cu at (243.0, 151.1)
- added C21: 47.0uF, Capacitor_THT:CP_Radial_D5.0mm_P2.00mm, F.Cu at (154.9, 136.3)
- added C21: 0.022, Capacitor_SMD:C_0805_2012Metric_Pad1.18x1.45mm_HandSolder, F.Cu at (168.3, 104.1)
- added C22: 0.1, Capacitor_SMD:C_0805_2012Metric_Pad1.18x1.45mm_HandSolder, B.Cu at (386.7, 160.0)
- added C23: 10.0, Capacitor_THT:CP_Radial_D4.0mm_P1.50mm, F.Cu at (391.9, 106.3)
- added C24: 1.0uF, Capacitor_SMD:C_0805_2012Metric_Pad1.18x1.45mm_HandSolder, F.Cu at (151.3, 95.2)
- added C6: 0.1, Capacitor_SMD:C_0805_2012Metric_Pad1.18x1.45mm_HandSolder, F.Cu at (163.8, 111.1)
- added C7: 6800, Capacitor_SMD:C_0805_2012Metric_Pad1.18x1.45mm_HandSolder, F.Cu at (157.5, 87.6)
- added C8: 47.0, Capacitor_THT:CP_Radial_D5.0mm_P2.50mm, F.Cu at (222.9, 85.5)
- added C9: 1.0uF, Capacitor_SMD:C_0805_2012Metric_Pad1.18x1.45mm_HandSolder, F.Cu at (170.8, 99.7)
- added D2: D, Diode_SMD:D_1206_3216Metric_Pad1.42x1.75mm_HandSolder, F.Cu at (348.9, 90.3)
- added D3: D, Diode_SMD:D_1206_3216Metric_Pad1.42x1.75mm_HandSolder, B.Cu at (217.7, 94.1)
- added D4: INT, LED_THT:LED_D2.0mm_W4.8mm_H2.5mm_FlatTop, F.Cu at (194.3, 99.1)
- added D5: 1N4148W, Diode_SMD:D_SOD-123, F.Cu at (382.5, 80.8)
- added DD2: TZT_RP2040, Library:RP2040_purple_allPin, F.Cu at (202.1, 89.0)
- added FB2: FerriteBead_Small, Inductor_SMD:L_0805_2012Metric_Pad1.15x1.40mm_HandSolder, F.Cu at (258.9, 94.0)
- added J11: Conn_02x20_Odd_Even, Connector_PinSocket_2.54mm:PinSocket_2x20_P2.54mm_Vertical, F.Cu at (113.0, 114.3)
- added J12: Conn_02x20_Odd_Even, Library:EDGE_2x20, F.Cu at (277.1, 114.3)
- added J13: IN, Library:PJ320D_3.5mm_Jack, F.Cu at (173.9, 114.3)
- added J14: Conn_02x20_Odd_Even, Library:EDGE_2x20, F.Cu at (321.4, 114.4)
- added J15: Conn_02x10_Odd_Even, Library:EDGE_2x10, F.Cu at (144.3, 81.3)
- added J16: Conn_02x20_Odd_Even, Library:EDGE_2x20, F.Cu at (144.4, 114.3)
- added J17: Conn_02x10_Odd_Even, Connector_PinSocket_2.54mm:PinSocket_2x10_P2.54mm_Vertical, F.Cu at (113.0, 81.3)
- added J18: Conn_02x10_Odd_Even, Library:EDGE_2x10, F.Cu at (277.1, 81.2)
- added J19: VGA, Connector_Dsub:DSUB-15-HD_Female_Horizontal_P2.29x1.98mm_EdgePinOffset3.03mm_Housed_MountingHolesOffset4.94mm, F.Cu at (206.1, 78.1)
- added J20: Micro_SD_Card, Library:GCT-MEM2055-00-190-01-A, F.Cu at (64.6, 86.5)
- added J22: PJ320D, Library:PJ320D_3.5mm_Jack, F.Cu at (262.5, 85.9)
- added J23: Conn_02x10_Odd_Even, Library:EDGE_2x10, F.Cu at (364.2, 81.3)
- added J24: Conn_02x10_Odd_Even, Library:EDGE_2x10, F.Cu at (232.8, 81.3)
- added J25: Conn_02x20_Odd_Even, Library:EDGE_2x20, F.Cu at (232.9, 114.4)
- added J26: Conn_02x10_Odd_Even, Library:EDGE_2x10, F.Cu at (188.4, 81.3)
- added J27: Conn_02x20_Odd_Even, Library:EDGE_2x20, F.Cu at (188.3, 114.4)
- added J28: OUT, Library:PJ320D_3.5mm_Jack, F.Cu at (173.9, 85.7)
- added J29: Conn_02x10_Odd_Even, Connector_PinSocket_2.54mm:PinSocket_2x10_P2.54mm_Vertical, F.Cu at (91.4, 81.3)
- added J30: Conn_02x20_Odd_Even, Connector_PinSocket_2.54mm:PinSocket_2x20_P2.54mm_Vertical, F.Cu at (91.4, 114.3)
- added J31: Conn_02x20_Odd_Even, Library:EDGE_2x20, F.Cu at (364.2, 114.3)
- added J5: Conn_02x10_Odd_Even, Library:EDGE_2x10, F.Cu at (321.4, 81.2)
- added J6: Conn_02x20_Odd_Even, Connector_PinSocket_2.54mm:PinSocket_2x20_P2.54mm_Vertical, F.Cu at (134.6, 114.3)
- added J9: Conn_02x10_Odd_Even, Connector_PinSocket_2.54mm:PinSocket_2x10_P2.54mm_Vertical, F.Cu at (134.7, 81.3)
- added JP1: Jumper_2_Small_Open, Connector_PinHeader_2.54mm:PinHeader_1x02_P2.54mm_Vertical, F.Cu at (198.8, 101.6)
- added JP2: Jumper_2_Small_Open, Connector_PinHeader_2.54mm:PinHeader_1x02_P2.54mm_Vertical, F.Cu at (198.8, 106.7)
- added JP3: Jumper_2_Small_Open, Connector_PinHeader_2.54mm:PinHeader_1x02_P2.54mm_Vertical, F.Cu at (198.8, 116.8)
- added JP4: Jumper_2_Small_Open, Connector_PinHeader_2.54mm:PinHeader_1x02_P2.54mm_Vertical, F.Cu at (198.8, 114.3)
- added JP5: Jumper_2_Small_Open, Connector_PinHeader_2.54mm:PinHeader_1x02_P2.54mm_Vertical, F.Cu at (198.8, 129.5)
- added JP6: Jumper_2_Small_Open, Connector_PinHeader_2.54mm:PinHeader_1x02_P2.54mm_Vertical, F.Cu at (198.8, 124.5)
- added JP7: Jumper_2_Small_Open, Connector_PinHeader_2.54mm:PinHeader_1x02_P2.54mm_Vertical, F.Cu at (198.8, 91.4)
- added JP8: Jumper_2_Small_Open, Connector_PinHeader_2.54mm:PinHeader_1x02_P2.54mm_Vertical, F.Cu at (198.8, 94.0)
- added Q2: BC817, Package_TO_SOT_SMD:SOT-23, F.Cu at (374.0, 80.0)
- added R1: 1k, Resistor_SMD:R_0805_2012Metric_Pad1.20x1.40mm_HandSolder, F.Cu at (163.8, 95.2)
- added R17: 4.7k, Resistor_SMD:R_0805_2012Metric_Pad1.20x1.40mm_HandSolder, F.Cu at (305.0, 149.8)
- added R18: 4.7k, Resistor_SMD:R_0805_2012Metric_Pad1.20x1.40mm_HandSolder, F.Cu at (305.0, 154.9)
- added R19: 4.7k, Resistor_SMD:R_0805_2012Metric_Pad1.20x1.40mm_HandSolder, F.Cu at (305.0, 160.0)
- added R23: 3.6k, Resistor_SMD:R_0805_2012Metric_Pad1.20x1.40mm_HandSolder, F.Cu at (174.0, 104.1)
- added R24: 10k, Resistor_SMD:R_0805_2012Metric_Pad1.20x1.40mm_HandSolder, F.Cu at (344.2, 127.0)
- added R25: 4,7k, Resistor_SMD:R_0805_2012Metric_Pad1.20x1.40mm_HandSolder, F.Cu at (385.4, 88.4)
- added R26: 100, Resistor_SMD:R_0805_2012Metric_Pad1.20x1.40mm_HandSolder, F.Cu at (244.1, 157.9)
- added R27: 100, Resistor_SMD:R_0805_2012Metric_Pad1.20x1.40mm_HandSolder, F.Cu at (162.2, 154.1)
- added R28: 1k, Resistor_SMD:R_0805_2012Metric_Pad1.20x1.40mm_HandSolder, F.Cu at (369.6, 88.9)
- added R28: 4.7k, Resistor_SMD:R_0805_2012Metric_Pad1.20x1.40mm_HandSolder, F.Cu at (168.3, 99.7)
- added R29: 51, Resistor_SMD:R_0805_2012Metric_Pad1.20x1.40mm_HandSolder, F.Cu at (382.0, 77.6)
- added R30: 330, Resistor_SMD:R_0805_2012Metric_Pad1.20x1.40mm_HandSolder, F.Cu at (368.9, 129.5)
- added R31: 330, Resistor_SMD:R_0805_2012Metric_Pad1.20x1.40mm_HandSolder, F.Cu at (368.9, 132.1)
- added R32: 330, Resistor_SMD:R_0805_2012Metric_Pad1.20x1.40mm_HandSolder, B.Cu at (368.9, 134.6)
- added R33: 330, Resistor_SMD:R_0805_2012Metric_Pad1.20x1.40mm_HandSolder, B.Cu at (368.9, 132.1)
- added R34: 3.9k, Resistor_SMD:R_0805_2012Metric_Pad1.20x1.40mm_HandSolder, B.Cu at (210.2, 96.6)
- added R35: 1k, Resistor_SMD:R_0805_2012Metric_Pad1.20x1.40mm_HandSolder, B.Cu at (210.2, 101.7)
- added R36: 3.9k, Resistor_SMD:R_0805_2012Metric_Pad1.20x1.40mm_HandSolder, B.Cu at (210.2, 109.3)
- added R37: 1k, Resistor_SMD:R_0805_2012Metric_Pad1.20x1.40mm_HandSolder, B.Cu at (210.2, 114.4)
- added R38: 3.9k, Resistor_SMD:R_0805_2012Metric_Pad1.20x1.40mm_HandSolder, B.Cu at (210.2, 119.5)
- added R39: 1k, Resistor_SMD:R_0805_2012Metric_Pad1.20x1.40mm_HandSolder, B.Cu at (210.2, 124.6)
- added R40: 2k, Resistor_SMD:R_0805_2012Metric_Pad1.20x1.40mm_HandSolder, B.Cu at (210.2, 99.2)
- added R41: 510, Resistor_SMD:R_0805_2012Metric_Pad1.20x1.40mm_HandSolder, B.Cu at (210.2, 106.8)
- added R42: 2k, Resistor_SMD:R_0805_2012Metric_Pad1.20x1.40mm_HandSolder, B.Cu at (210.2, 111.9)
- added R43: 510, Resistor_SMD:R_0805_2012Metric_Pad1.20x1.40mm_HandSolder, B.Cu at (210.2, 117.0)
- added R44: 2k, Resistor_SMD:R_0805_2012Metric_Pad1.20x1.40mm_HandSolder, B.Cu at (210.2, 122.0)
- added R45: 510, Resistor_SMD:R_0805_2012Metric_Pad1.20x1.40mm_HandSolder, B.Cu at (210.2, 129.7)
- added R46: 100, Resistor_SMD:R_0805_2012Metric_Pad1.20x1.40mm_HandSolder, B.Cu at (210.2, 91.6)
- added R47: 100, Resistor_SMD:R_0805_2012Metric_Pad1.20x1.40mm_HandSolder, B.Cu at (210.2, 94.1)
- added R48: 1k, Resistor_SMD:R_0805_2012Metric_Pad1.20x1.40mm_HandSolder, B.Cu at (193.0, 104.1)
- added R49: 330, Resistor_SMD:R_0805_2012Metric_Pad1.20x1.40mm_HandSolder, B.Cu at (368.9, 129.6)
- added R50: 330, Resistor_SMD:R_0805_2012Metric_Pad1.20x1.40mm_HandSolder, F.Cu at (368.9, 134.6)
- added R51: 330, Resistor_SMD:R_0805_2012Metric_Pad1.20x1.40mm_HandSolder, F.Cu at (375.0, 124.5)
- added R52: 330, Resistor_SMD:R_0805_2012Metric_Pad1.20x1.40mm_HandSolder, F.Cu at (375.0, 127.0)
- added R53: 4,7k, Resistor_SMD:R_0805_2012Metric_Pad1.20x1.40mm_HandSolder, B.Cu at (383.9, 116.8)
- added R54: 4,7k, Resistor_SMD:R_0805_2012Metric_Pad1.20x1.40mm_HandSolder, B.Cu at (383.9, 142.2)
- added R55: 1k, Resistor_SMD:R_0805_2012Metric_Pad1.20x1.40mm_HandSolder, B.Cu at (383.9, 137.2)
- added SW1: "RESET", Button_Switch_THT:SW_Tactile_SPST_Angled_PTS645Vx31-2LFS, F.Cu at (355.5, 93.0)
- added SW2: "RESET", Button_Switch_THT:SW_Tactile_SPST_Angled_PTS645Vx31-2LFS, F.Cu at (311.4, 93.2)
- added U10: 74LS74, Package_SO:SOIC-14_3.9x8.7mm_P1.27mm, F.Cu at (377.8, 98.9)
- added U11: 8086_Min_Mode, Package_DIP:DIP-40_W15.24mm, F.Cu at (395.0, 160.0)
- added U12: 74LS08, Package_SO:SOIC-14_3.9x8.7mm_P1.27mm, F.Cu at (378.0, 88.8)
- added U5: LM1117MP-3.3, Package_TO_SOT_SMD:SOT-223-3_TabPin2, F.Cu at (48.3, 136.5)
- added U7: SN76489AN, Package_DIP:DIP-16_W7.62mm_LongPads, F.Cu at (243.0, 124.5)
- added U8: 74LS74, Package_SO:SOIC-14_3.9x8.7mm_P1.27mm, F.Cu at (154.3, 125.1)
- added U9: 74LS04, Package_SO:SOIC-14_3.9x8.7mm_P1.27mm, F.Cu at (390.8, 98.9)
- added USB1: TYPE-C-31-M-12, Library:USB-TYPE-C-31-M-12_lib2, B.Cu at (38.3, 91.5)
- added u1: ~, Library:RP2350B_WeAct, F.Cu at (40.3, 118.2)
- C1: value 6800 -> 0.1
- C3: value 0.1uF -> 0.022
- J10: value VGA -> NES_Joystick1; footprint Connector_Dsub:DSUB-15-HD_Female_Horizontal_P2.29x1.98mm_EdgePinOffset3.03mm_Housed_MountingHolesOffset4.94mm -> Connector_Dsub:DSUB-9_Male_Horizontal_P2.77x2.84mm_EdgePinOffset4.94mm_Housed_MountingHolesOffset7.48mm
- J7: footprint Connector_Dsub:DSUB-9_Male_Vertical_P2.77x2.84mm_MountingHoles -> Connector_Dsub:DSUB-9_Male_Horizontal_P2.77x2.84mm_EdgePinOffset4.94mm_Housed_MountingHolesOffset7.48mm
- J8: value NES_Joystick2 -> +5=Vbus; footprint Connector_Dsub:DSUB-9_Male_Vertical_P2.77x2.84mm_MountingHoles -> Connector_PinHeader_2.54mm:PinHeader_1x02_P2.54mm_Vertical
- R10, R14: value 510 -> 100
- R11: value 2k -> 3.6k
- R12: value 510 -> 4.7k
- R13: value 2k -> 1k
- R15, R16: value 100 -> 3.6k
- R3: value 3.9k -> 1k
- R4: value 1k -> 5.1K; moved to B.Cu
- R5: value 3.9k -> 5.1K; moved to B.Cu
- R6, R8: value 1k -> 4.7k
- R7: value 3.9k -> 100k
- R9: value 2k -> 100k
- U2: value SN76489AN -> LM393; footprint Package_DIP:DIP-16_W7.62mm_LongPads -> Package_SO:SOIC-8_3.9x4.9mm_P1.27mm
- moved R21 238.0 mm to (349.3, 119.3)
- moved U4 234.5 mm to (353.4, 162.6), turned to 180 degrees
- moved C5 233.9 mm to (344.2, 137.1), turned to 180 degrees
- moved R20 233.6 mm to (344.2, 124.4), turned to 180 degrees
- moved R22 232.9 mm to (344.2, 121.9), turned to 180 degrees
- moved C4 231.1 mm to (307.3, 166.9)
- moved R3 187.7 mm to (253.8, 94.0), turned to 90 degrees
- moved U3 174.0 mm to (310.1, 162.5), turned to 180 degrees
- moved J10 161.1 mm to (249.4, 163.4)
- moved J8 143.6 mm to (41.9, 163.8), turned to 90 degrees
- moved J7 118.1 mm to (160.8, 163.4)
- moved J1 117.7 mm to (41.9, 157.8), turned to 90 degrees
- moved J2 115.7 mm to (41.9, 154.9), turned to 90 degrees
- moved J4 101.9 mm to (41.9, 119.7), turned to 90 degrees
- moved J3 101.4 mm to (41.9, 121.9), turned to 90 degrees
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Connections:
- C1 pad 1: Net-(C1-Pad1) -> VCC_MSX
- C1 pad 2: GND -> GND_MSX
- C2 pad 2: Net-(C1-Pad1) -> /IO_MSX/SAVE_MSX
- C3 pad 1: GND -> Net-(C3-Pad1)
- C3 pad 2: +5V -> GND_MSX
- FB1 pad 1: Net-(C2-Pad1) -> Net-(C17-Pad1)
- J1 pad 1: GND -> /VBUS
- J1 pad 10: /GP35 -> /GP13
- J1 pad 11: /GP33 -> /GP15
- J1 pad 12: /GP31 -> /GP17
- J1 pad 13: /D7 -> /GP19
- J1 pad 14: /D5 -> /GP21
- J1 pad 15: /D3 -> /GP23
- J1 pad 2: /EN -> GND
- J1 pad 3: /3V3 -> /VREF
- J1 pad 4: /Encoder_B -> /GP1
- J1 pad 5: /GP45 -> /GP3
- J1 pad 6: /GP43 -> /GP5
- J1 pad 7: /GP41 -> /GP7
- J1 pad 8: /GP39 -> /GP9
- J1 pad 9: /GP37 -> /GP11
- J10 pad 0: GND -> GND_IO
- J10 pad 1: /R -> /I0_SG1000/JOY_DATA2
- J10 pad 2: /G -> /I0_SG1000/JOY_DATA1
- J10 pad 3: /B -> /I0_SG1000/JOY_LATCH
- J10 pad 4: unconnected-(J10-Pad4) -> /I0_SG1000/JOY_CLK
- J10 pad 5: GND -> unconnected-(J10-Pad5)
- J10 pad 6: GND -> Net-(J10-Pad6)
- J10 pad 7: GND -> unconnected-(J10-Pad7)
- J10 pad 8: GND -> /I0_SG1000/GND
- J2 pad 1: GND -> /+5V
- J2 pad 10: /GP36 -> /GP14
- J2 pad 11: /GP34 -> /GP16
- J2 pad 12: /GP32 -> /GP18
- J2 pad 13: /GP30 -> /GP20
- J2 pad 14: /D6 -> /GP22
- J2 pad 15: /D4 -> /GP24
- J2 pad 3: /3V3 -> /GP0
- J2 pad 4: /RUN -> /GP2
- J2 pad 5: /Encoder_A -> /GP4
- J2 pad 6: /GP44 -> /GP6
- J2 pad 7: /GP42 -> /GP8
- J2 pad 8: /GP40 -> /GP10
- J2 pad 9: /GP38 -> /GP12
- J3 pad 1: /VBUS -> GND
- J3 pad 10: /GP13 -> /GP35
- J3 pad 11: /GP15 -> /GP33
- J3 pad 12: /GP17 -> /GP31
- J3 pad 13: /GP19 -> /GP29
- J3 pad 14: /GP21 -> /GP27
- J3 pad 15: /D1 -> /GP25
- J3 pad 2: GND -> /EN
- J3 pad 3: /VREF -> +3.3V
- J3 pad 4: /GP1 -> /GP47
- J3 pad 5: /GP3 -> /GP45
- J3 pad 6: /GP5 -> /GP43
- J3 pad 7: /GP7 -> /GP41
- J3 pad 8: /GP9 -> /GP39
- J3 pad 9: /GP11 -> /GP37
- J4 pad 1: /5V -> GND
- J4 pad 10: /GP14 -> /GP36
- J4 pad 11: /GP16 -> /GP34
- J4 pad 12: /GP18 -> /GP32
- J4 pad 13: /GP20 -> /GP30
- J4 pad 14: /D0 -> /GP28
- J4 pad 15: /D2 -> /GP26
- J4 pad 3: /GP0 -> +3.3V
- J4 pad 4: /GP2 -> /RUN
- J4 pad 5: /GP4 -> /GP46
- J4 pad 6: /A0 -> /GP44
- J4 pad 7: /GP8 -> /GP42
- J4 pad 8: /GP10 -> /GP40
- J4 pad 9: /GP12 -> /GP38
- J7 pad 0: GND -> GND_MSX
- J7 pad 1: unconnected-(J7-Pad1) -> /IO_MSX/JOY_DATA2_MSX
- J7 pad 2: /GP44 -> /IO_MSX/JOY_DATA1_MSX
- J7 pad 3: /GP43 -> /IO_MSX/JOY_LATCH_MSX
- J7 pad 4: /GP42 -> /IO_MSX/JOY_CLK_MSX
- J7 pad 6: /5V -> Net-(J7-Pad6)
- J7 pad 8: GND -> GND_MSX
- J8 pad 1: unconnected-(J8-Pad1) -> /VBUS
- J8 pad 2: /GP45 -> /+5V
- R10 pad 1: Net-(DD1-GP5) -> TAPE_OUT
- R10 pad 2: /R -> GND_MSX
- R11 pad 1: Net-(DD1-GP7) -> /IO_MSX/3V3
- R11 pad 2: /G -> /IO_MSX/Tape_In
- R12 pad 2: /G -> VCC_MSX
- R13 pad 1: Net-(DD1-GP11) -> /IO_MSX/OUT_PWM_MSX
- R13 pad 2: /B -> Net-(C17-Pad2)
- R14 pad 1: Net-(DD1-GP13) -> Net-(C24-Pad1)
- R14 pad 2: /B -> Net-(U2A-+)
- R15 pad 1: Net-(J10-Pad13) -> Net-(J13-T)
- R15 pad 2: /HSYNC -> Net-(C19-Pad1)
- R16 pad 1: Net-(J10-Pad14) -> Net-(C19-Pad1)
- R16 pad 2: /VSYNC -> Net-(C9-Pad2)
- R2 pad 1: /Audio_Out -> GND_MSX
- R2 pad 2: Net-(C1-Pad1) -> Net-(C24-Pad1)
- R3 pad 1: Net-(DD1-GP2) -> /I0_SG1000/Audio_Out
- R3 pad 2: /R -> Net-(C12-Pad1)
- R4 pad 1: Net-(DD1-GP4) -> GND
- R4 pad 2: /R -> Net-(USB1-CC1)
- R5 pad 1: Net-(DD1-GP6) -> GND
- R5 pad 2: /G -> Net-(USB1-CC2)
- R6 pad 1: Net-(DD1-GP8) -> Net-(C2-Pad1)
- R6 pad 2: /G -> Net-(C3-Pad1)
- R7 pad 1: Net-(DD1-GP10) -> Net-(C24-Pad1)
- R7 pad 2: /B -> Net-(U2A--)
- R8 pad 1: Net-(DD1-GP12) -> Net-(C3-Pad1)
- R8 pad 2: /B -> TAPE_OUT
- R9 pad 1: Net-(DD1-GP3) -> Net-(U2A-+)
- R9 pad 2: /R -> /IO_MSX/Tape_In
- U2 pad 1: /D5 -> /IO_MSX/Tape_In
- U2 pad 2: /D6 -> Net-(U2A--)
- U2 pad 3: /D7 -> Net-(U2A-+)
- U2 pad 4: /GP35 -> GND_MSX
- U2 pad 5: /GP35 -> GND_MSX
- U2 pad 6: /GP41 -> GND_MSX
- U2 pad 7: /Audio_Out -> unconnected-(U2-Pad7)
- U2 pad 8: GND -> VCC_MSX
- U3 pad 37: /MOC6502/CLK -> /MOC6502/CLK6502
- U4 pad 26: /Z80/~{RESET} -> Net-(D2-A)
Routing:
- net GND: track 0.00 -> 341.1 mm
- net GND_MSX: track 0.00 -> 338.3 mm, vias 0 -> 2
- net GND_IO: track 0.00 -> 282.1 mm, vias 0 -> 3
- net VCC86: track 0.00 -> 273.2 mm, vias 0 -> 2
- net GND86: track 0.00 -> 207.2 mm, vias 0 -> 4
- net GND1: track 0.00 -> 206.7 mm, vias 0 -> 3
- net /+5V: track 0.00 -> 205.9 mm, vias 0 -> 3
- net GND_VDP: track 0.00 -> 188.2 mm, vias 0 -> 3
- net +3.3V: track 0.00 -> 147.0 mm, vias 0 -> 1
- net GND2: track 0.00 -> 132.6 mm, vias 0 -> 2
- net VCC_VDP: track 0.00 -> 121.3 mm, vias 0 -> 1
- net /GP43: track 0.00 -> 113.4 mm, vias 0 -> 1
- net /GP41: track 0.00 -> 112.6 mm, vias 0 -> 1
- net /GP47: track 0.00 -> 110.8 mm
- net /GP45: track 0.00 -> 106.6 mm
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- added copper zone on B.Cu, net GND
- added copper zone on F.Cu, net GND
Other:
- board outline added: 363.4 x 100.1 mm
- board text added: "+3.3V"
- board text added: "6502CPU"
- board text added: "74LS04"
- board text added: "74LS08"
- board text added: "74LS74"
- board text added: "8086"
- board text added: "GND"
- board text added: "GP0"
- board text added: "GP1"
- board text added: "GP10"
- board text added: "GP11"
- board text added: "GP12"
- board text added: "GP13"
- board text added: "GP14"
- board text added: "GP15"
- board text added: "GP16"
- board text added: "GP17"
- board text added: "GP18"
- board text added: "GP19"
- board text added: "GP2"
- board text added: "GP20"
- board text added: "GP21"
- board text added: "GP22"
- board text added: "GP23"
- board text added: "GP24"
- board text added: "GP25"
- board text added: "GP26"
- board text added: "GP27"
- board text added: "GP28"
- board text added: "GP29"
- board text added: "GP3"
- board text added: "GP30"
- board text added: "GP31"
- board text added: "GP32"
- board text added: "GP33"
- board text added: "GP34"
- board text added: "GP35"
- board text added: "GP36"
- board text added: "GP37"
- board text added: "GP38"
- board text added: "GP39"
- board text added: "GP4"
- board text added: "GP40"
- board text added: "GP41"
- board text added: "GP42"
- board text added: "GP43"
- board text added: "GP44"
- board text added: "GP45"
- board text added: "GP46"
- board text added: "GP47"
- board text added: "GP5"
- board text added: "GP6"
- board text added: "GP7"
- board text added: "GP8"
- board text added: "GP9"
- board text added: "IN"
- board text added: "J17"
- board text added: "MSX"
- board text added: "OUT"
- board text added: "RESET"
- board text added: "RP2350B"
- board text added: "SG1000/COLECO"
- board text added: "VDP PICO9918"
- board text added: "Z80CPU"

Commit message: Update RP2350B_Consol.kicad_pcb
Connections:
- J24 pad 5: unconnected-(J24-Pin_5-Pad5) -> /I0_SG1000/~{WAIT_PSG}
- J25 pad 9: /I0_SG1000/~{WAIT_PSG} -> unconnected-(J25-Pin_9-Pad9)
- J5 pad 5: unconnected-(J5-Pin_5-Pad5) -> /Z80/~{WAIT}
Routing:
- net /Z80/~{WAIT}: track 23.0 -> 70.4 mm, vias 0 -> 1
- net /I0_SG1000/~{WAIT_PSG}: track 30.9 -> 62.7 mm, vias 0 -> 1
