File: IO_SG1000.kicad_sch (KiCad schematic)
At the start: 12 parts, among them J10 NES_Joystick1, J22 PJ320D, J24 Conn_02x10_Odd_Even, J25 Conn_02x20_Odd_Even, U7 SN76489AN

Commit message: Update IO_SG1000.kicad_sch
Connections:
- net ~{WAIT_PSG}: now also J24.5 (Pin_5); no longer J25.9 (Pin_9)
Changed lines of the file:
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@@
+	(wire
+		(pts
+			(xy 36.83 29.21) (xy 44.45 29.21)
+		)
+		(stroke
+			(width 0)
+			(type default)
+		)
+	)
 	(wire
 		(pts
@@
 	(wire
 		(pts
+			(xy 62.23 26.67) (xy 57.15 26.67)
+		)
+		(stroke
+			(width 0)
+			(type default)
+		)
+	)
+	(wire
+		(pts
 			(xy 213.36 45.72) (xy 215.9 45.72)
 		)
@@
 	(wire
 		(pts
-			(xy 62.23 26.67) (xy 57.15 26.67)
-		)
-		(stroke
-			(width 0)
-			(type default)
-		)
-	)
-	(wire
-		(pts
 			(xy 214.63 80.01) (xy 218.44 80.01)
 		)
@@
 		(pts
 			(xy 255.27 33.02) (xy 259.08 33.02)
-		)
-		(stroke
-			(width 0)
-			(type default)
-		)
-	)
-	(wire
-		(pts
-			(xy 36.83 66.04) (xy 44.45 66.04)
 		)
 		(stroke
@@
 	)
 	(label "~{WAIT_PSG}"
-		(at 36.83 66.04 180)
-		(fields_autoplaced yes)
-		(effects
+		(at 36.83 29.21 180)
+		(fields_autoplaced yes)
+		(effects
