File: plates/Z80/z80/z80.kicad_pcb (KiCad board)
At the start: 2 copper layers, 40 x 100 mm, 90 parts, among them J14 Conn_02x20_Odd_Even, J5 Conn_02x10_Odd_Even, SW1 "RESET", U4 Z80CPU

Commit message: Update z80.kicad_pcb
Parts:
- removed the ? at (124.7, 66.8)
- removed the ? at (134.8, 59.1)
- removed the ? at (134.8, 76.9)
- removed the ? at (122.1, 61.7)
- removed the ? at (134.8, 71.8)
- removed the ? at (122.1, 71.8)
- removed the ? at (132.3, 74.4)
- removed the ? at (137.4, 59.1)
- removed the ? at (122.1, 66.8)
- removed the ? at (132.3, 76.9)
- removed the ? at (124.7, 71.8)
- removed the ? at (124.7, 59.1)
- removed the ? at (134.8, 66.8)
- removed the ? at (137.4, 69.3)
- removed the ? at (137.4, 61.7)
- removed the ? at (127.2, 64.2)
- removed the ? at (137.4, 64.2)
- removed the ? at (127.2, 74.4)
- removed the ? at (127.2, 76.9)
- removed the ? at (124.7, 56.6)
- removed the ? at (129.8, 74.4)
- removed the ? at (132.3, 79.5)
- removed the ? at (129.8, 64.2)
- removed the ? at (139.9, 59.1)
- removed the ? at (139.9, 71.8)
- removed the ? at (122.1, 56.6)
- removed the ? at (124.7, 79.5)
- removed the ? at (137.4, 76.9)
- removed the ? at (124.7, 64.2)
- removed the ? at (134.8, 64.2)
- removed the ? at (139.9, 56.6)
- removed the ? at (132.3, 59.1)
- removed the ? at (124.7, 61.7)
- removed the ? at (132.3, 71.8)
- removed the ? at (134.8, 79.5)
- removed the ? at (127.2, 59.1)
- removed the ? at (137.4, 79.5)
- removed the ? at (139.9, 61.7)
- removed the ? at (122.1, 69.3)
- removed the ? at (127.2, 61.7)
- removed the ? at (139.9, 66.8)
- removed the ? at (139.9, 79.5)
- removed the ? at (139.9, 64.2)
- removed the ? at (132.3, 69.3)
- removed the ? at (132.3, 61.7)
- removed the ? at (137.4, 66.8)
- removed the ? at (134.8, 61.7)
- removed the ? at (132.3, 56.6)
- removed the ? at (129.8, 71.8)
- removed the ? at (127.2, 71.8)
- removed the ? at (122.1, 64.2)
- removed the ? at (139.9, 74.4)
- removed the ? at (129.8, 76.9)
- removed the ? at (127.2, 79.5)
- removed the ? at (139.9, 69.3)
- removed the ? at (124.7, 74.4)
- removed the ? at (139.9, 76.9)
- removed the ? at (137.4, 74.4)
- removed the ? at (124.7, 76.9)
- removed the ? at (132.3, 66.8)
- removed the ? at (129.8, 79.5)
- removed the ? at (127.2, 66.8)
- removed the ? at (122.1, 59.1)
- removed the ? at (137.4, 71.8)
- removed the ? at (124.7, 69.3)
- removed the ? at (134.8, 74.4)
- removed the ? at (137.4, 56.6)
- removed the ? at (134.8, 56.6)
- removed the ? at (122.1, 76.9)
- removed the ? at (132.3, 64.2)
- removed the ? at (129.8, 59.1)
- removed the ? at (134.8, 69.3)
- removed the ? at (127.2, 69.3)
- removed the ? at (129.8, 66.8)
- removed the ? at (129.8, 61.7)
- removed the ? at (129.8, 69.3)
- removed the ? at (129.8, 56.6)
- removed the ? at (122.1, 74.4)
- removed the ? at (127.2, 56.6)
- removed the ? at (122.1, 79.5)
- added ?: , , F.Cu at (149.7, 54.8)
- added ?: , , F.Cu at (134.5, 59.9)
- added ?: , , F.Cu at (144.6, 70.1)
- added ?: , , F.Cu at (144.6, 75.1)
- added ?: , , F.Cu at (137.0, 70.1)
- added ?: , , F.Cu at (144.6, 52.3)
- added ?: , , F.Cu at (142.1, 54.8)
- added ?: , , F.Cu at (131.9, 67.5)
- added ?: , , F.Cu at (147.2, 62.4)
- added ?: , , F.Cu at (131.9, 75.1)
- added ?: , , F.Cu at (139.6, 75.1)
- added ?: , , F.Cu at (139.6, 62.4)
- added ?: , , F.Cu at (134.5, 52.3)
- added ?: , , F.Cu at (131.9, 59.9)
- added ?: , , F.Cu at (137.0, 59.9)
- added ?: , , F.Cu at (142.1, 59.9)
- added ?: , , F.Cu at (134.5, 54.8)
- added ?: , , F.Cu at (144.6, 54.8)
- added ?: , , F.Cu at (134.5, 62.4)
- added ?: , , F.Cu at (149.7, 75.1)
- added ?: , , F.Cu at (137.0, 52.3)
- added ?: , , F.Cu at (131.9, 52.3)
- added ?: , , F.Cu at (137.0, 57.4)
- added ?: , , F.Cu at (134.5, 75.1)
- added ?: , , F.Cu at (149.7, 52.3)
- added ?: , , F.Cu at (144.6, 72.6)
- added ?: , , F.Cu at (147.2, 57.4)
- added ?: , , F.Cu at (147.2, 59.9)
- added ?: , , F.Cu at (144.6, 59.9)
- added ?: , , F.Cu at (149.7, 59.9)
- added ?: , , F.Cu at (139.6, 70.1)
- added ?: , , F.Cu at (149.7, 62.4)
- added ?: , , F.Cu at (147.2, 72.6)
- added ?: , , F.Cu at (144.6, 57.4)
- added ?: , , F.Cu at (142.1, 75.1)
- added ?: , , F.Cu at (147.2, 70.1)
- added ?: , , F.Cu at (139.6, 52.3)
- added ?: , , F.Cu at (147.2, 65.0)
- added ?: , , F.Cu at (137.0, 62.4)
- added ?: , , F.Cu at (147.2, 52.3)
- added ?: , , F.Cu at (139.6, 67.5)
- added ?: , , F.Cu at (131.9, 57.4)
- added ?: , , F.Cu at (149.7, 72.6)
- added ?: , , F.Cu at (131.9, 72.6)
- added ?: , , F.Cu at (147.2, 54.8)
- added ?: , , F.Cu at (149.7, 57.4)
- added ?: , , F.Cu at (149.7, 70.1)
- added ?: , , F.Cu at (142.1, 70.1)
- added ?: , , F.Cu at (131.9, 62.4)
- added ?: , , F.Cu at (134.5, 70.1)
- added ?: , , F.Cu at (139.6, 59.9)
- added ?: , , F.Cu at (137.0, 65.0)
- added ?: , , F.Cu at (144.6, 67.5)
- added ?: , , F.Cu at (139.6, 57.4)
- added ?: , , F.Cu at (137.0, 75.1)
- added ?: , , F.Cu at (137.0, 54.8)
- added ?: , , F.Cu at (131.9, 54.8)
- added ?: , , F.Cu at (134.5, 57.4)
- added ?: , , F.Cu at (142.1, 65.0)
- added ?: , , F.Cu at (139.6, 65.0)
- added ?: , , F.Cu at (139.6, 54.8)
- added ?: , , F.Cu at (137.0, 67.5)
- added ?: , , F.Cu at (142.1, 67.5)
- added ?: , , F.Cu at (149.7, 65.0)
- added ?: , , F.Cu at (144.6, 62.4)
- added ?: , , F.Cu at (147.2, 75.1)
- added ?: , , F.Cu at (139.6, 72.6)
- added ?: , , F.Cu at (134.5, 65.0)
- added ?: , , F.Cu at (131.9, 70.1)
- added ?: , , F.Cu at (142.1, 52.3)
- added ?: , , F.Cu at (147.2, 67.5)
- added ?: , , F.Cu at (142.1, 72.6)
- added ?: , , F.Cu at (131.9, 65.0)
- added ?: , , F.Cu at (134.5, 72.6)
- added ?: , , F.Cu at (137.0, 72.6)
- added ?: , , F.Cu at (144.6, 65.0)
- added ?: , , F.Cu at (142.1, 62.4)
- added ?: , , F.Cu at (149.7, 67.5)
- added ?: , , F.Cu at (142.1, 57.4)
- added ?: , , F.Cu at (134.5, 67.5)
- moved D2 10.7 mm to (153.1, 57.6)
- moved R21 10.7 mm to (153.5, 86.6)
- moved J14 10.7 mm to (125.6, 81.6)
- moved J5 10.7 mm to (125.6, 48.5)
- moved C5 10.7 mm to (148.4, 104.4)
- moved R20 10.7 mm to (148.4, 91.7)
- moved R22 10.7 mm to (148.4, 89.1)
- moved R24 10.7 mm to (148.4, 94.2)
- moved SW1 10.7 mm to (159.7, 60.2)
- moved U4 10.7 mm to (157.6, 129.8)
Routing:
- net (no net): track 1580.2 -> 1627.7 mm, vias 21 -> 22
